Commit message: adding collision bodies to simple robot

File: mujoco_ros_control/model/simple_robot.urdf (robot description, URDF)
Before this commit: robot simple_robot, 2 links, 1 joints
Links:
- link ball: geometry collision sphere radius=0.05; visual sphere radius=0.05
- link base_link: geometry collision box size=1.0 1.0 0.05; visual box size=1.0 1.0 0.05
